File: hw/hdlcSpy/hdlcSpy.kicad_pcb (KiCad board)
At the start: 4 copper layers, 60 x 60 mm, 35 parts, among them J1 Conn_01x24_Pin, J2 Conn_01x09, U1 LM2936-5.0, U2 SN65HVD1782, U3 SN65HVD1782, U5 SN74LVC1G14DBV, U6 SN74LVC1G14DBV

Commit message: feat: cleanup schematic and pcb
Parts:
- R12: value 1K -> 10R
- R2, R3, R4, R5, R6, R7: value 1K -> 10K
- moved C5 8.58 mm to (105.6, 115.8), turned to 90 degrees
- moved C6 8.51 mm to (100.8, 115.8), turned to 90 degrees
- moved U1 0.30 mm to (103.2, 122.1)

Commit message: feat: sch and pcb done
Add some Datasheets
Parts:
- added C7: 100N, Capacitor_SMD:C_0603_1608Metric_Pad1.08x0.95mm_HandSolder, B.Cu at (115.7, 106.0)
- added J3: Micro_SD_Card_Det_Hirose_DM3AT, Connector_Card:microSD_HC_Hirose_DM3D-SF, F.Cu at (113.1, 104.8)
- J1: value Conn_01x24_Pin -> MODULBUS
- moved D2 19.5 mm to (118.0, 84.2)
- moved D3 19.5 mm to (115.5, 84.2)
- moved R16 19.5 mm to (118.0, 80.6)
- moved R17 19.5 mm to (115.5, 80.6)
- moved R18 14.0 mm to (115.4, 119.8)
- moved D4 13.9 mm to (115.4, 123.2)
- moved D1 12.4 mm to (113.1, 123.2)
- moved R15 12.4 mm to (113.1, 119.7)
- moved Z1 12.2 mm to (110.8, 127.5), turned to 0 degrees
- moved D5 10.2 mm to (116.8, 92.3)
- moved C5 1.35 mm to (106.4, 116.8), turned to 0 degrees
- moved R12 1.30 mm to (95.8, 122.2)
- moved C6 1.22 mm to (100.1, 116.8), turned to 180 degrees
- moved C4 0.24 mm to (81.6, 104.4)
- moved C3 0.17 mm to (77.3, 100.5)
Connections:
- A1 pad 14: unconnected-(A1-GPIO10-Pad14) -> /DAT0
- A1 pad 15: unconnected-(A1-GPIO11-Pad15)_1 -> /DAT1
- A1 pad 16: unconnected-(A1-GPIO12-Pad16) -> /DAT2
- A1 pad 17: unconnected-(A1-GPIO13-Pad17) -> /DAT3/CD
- A1 pad 19: Net-(A1-GPIO14) -> /CLK
- A1 pad 20: Net-(A1-GPIO15) -> /CMD
- A1 pad 21: unconnected-(A1-GPIO16-Pad21)_1 -> /SWA
- A1 pad 22: unconnected-(A1-GPIO17-Pad22) -> Net-(A1-GPIO17)
- A1 pad 24: unconnected-(A1-GPIO18-Pad24)_1 -> Net-(A1-GPIO18)
- R16 pad 1: Net-(A1-GPIO15) -> Net-(A1-GPIO17)
- R17 pad 1: Net-(A1-GPIO14) -> Net-(A1-GPIO18)
Routing:
- net GND: track 0.00 -> 63.3 mm, vias 0 -> 43
- net Net-(A1-VSYS): track 0.00 -> 59.7 mm
- net 5V-Ext: track 0.00 -> 43.6 mm, vias 0 -> 3
- net /DAT0: track 0.00 -> 42.9 mm, vias 0 -> 2
- net /DAT1: track 0.00 -> 40.6 mm
- net /SWA: track 0.00 -> 30.3 mm, vias 0 -> 1
- net /DAT2: track 0.00 -> 25.4 mm, vias 0 -> 2
- net /DAT3/CD: track 0.00 -> 24.5 mm, vias 0 -> 1
- net 3V3: track 0.00 -> 24.4 mm, vias 0 -> 13
- net /CLK: track 0.00 -> 21.2 mm
- net /Data+: track 0.00 -> 19.9 mm
- net /Clk_TX: track 0.00 -> 19.4 mm
- net /Data-: track 0.00 -> 16.5 mm
- net /CMD: track 0.00 -> 16.2 mm
- net /Clk-: track 0.00 -> 16.1 mm
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Other:
- board text added: "${COMPANY} ${PROJECTNAME} ${PROJECTNAME}-${PCB-Rev} ${CURRENT_DATE}"
- board text added: "Gnd"

Commit message: feat: orderd at Jjlcpcb
Parts:
- J1: value MODULBUS -> PIN HEADER 2.0MM PITCH STR SMT,2
- J2: value Conn_01x09 -> Connector_PinHeader_2.54mm:PinHeader_1x09_P2.54mm_Vertical
- U2, U3: value SN65HVD1782 -> ST4E1240DT
Changed lines of the file:
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@@
 			)
 		)
-		(property "Value" "SN65HVD1782"
+		(property "Value" "ST4E1240DT"
 			(at 0 3.4 90)
 			(layer "F.Fab")
@@
 			)
 		)
+		(property "DigiKey" "HR1972CT-ND"
+			(at 0 0 90)
+			(unlocked yes)
+			(layer "F.Fab")
+			(hide yes)
+			(effects
+				(font
+					(size 1 1)
+					(thickness 0.15)
+				)
+			)
+		)
 		(property ki_fp_filters "microSD*")
 		(sheetname "/")
@@
 			)
 		)
-		(property "Value" "SN65HVD1782"
+		(property "Value" "ST4E1240DT"
 			(at 0 3.4 90)
 			(layer "F.Fab")
@@
 			)
 		)
-		(property "Value" "MODULBUS"
+		(property "Value" "PIN HEADER 2.0MM PITCH STR SMT,2"
 			(at 0 13.11 90)
 			(layer "F.Fab")
@@
 			)
 		)
-		(property "DigiKey" ""
+		(property "DigiKey" "664-G825M24401YEUTR-ND"
 			(at 0 0 90)
 			(unlocked yes)
@@
 			)
 		)
-		(attr smd exclude_from_pos_files)
+		(attr smd)
 		(duplicate_pad_numbers_are_jumpers no)
 		(fp_line
@@
 			)
 		)
-		(attr through_hole)
+		(attr through_hole dnp)
 		(duplicate_pad_numbers_are_jumpers no)
 		(fp_line
@@
 			)
 		)
-		(property "Value" "Conn_01x09"
+		(property "Value" "Connector_PinHeader_2.54mm:PinHeader_1x09_P2.54mm_Vertical"
 			(at 0 22.7 90)
 			(layer "F.Fab")
@@
 			)
 		)
-		(attr smd)
+		(attr smd dnp)
 		(duplicate_pad_numbers_are_jumpers no)
 		(fp_line
